File: side.kicad_sch (KiCad schematic)
At the start: 45 parts, among them SW1 SW_SPST, SW10 SW_SPST, SW11 SW_SPST, SW12 SW_SPST, SW13 SW_SPST, SW14 SW_SPST, SW15 SW_SPST, SW16 SW_SPST, SW17 SW_SPST, SW18 SW_SPST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

Commit message: footprints
Parts:
- added H5, H6, H7: MountingHole, Panelization:mouse-bite-5mm-slot, symbol Mechanical:MountingHole
- added SW19: SW_SPDT, switch:SW-SMD_MSK12CO2, symbol Switch:SW_SPDT
- U1: footprint PCM_marbastlib-xp-promicroish:Xiao_nRF52840_ACH -> nrf52840:modified-XIAO-nRF52840-SMD
Connections:
- net at R2.2, U1.16 (BAT+): now also SW19.2 (B); no longer TP2.1
- new net: SW19.1 (A), TP2.1
Other:
- moved on the sheet: D1, D10, D11, D12, D13, D14, D15, D16, D17, D18, D2, D3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
