File: winglets.kicad_pcb (KiCad board)
At the start: 2 copper layers, 12.8 x 6.6 mm, 98 parts, among them SW1 SW_SPST, SW10 SW_SPST, SW11 SW_SPST, SW12 SW_SPST, SW13 SW_SPST, SW14 SW_SPST, SW15 SW_SPST, SW16 SW_SPST, SW17 SW_SPST, SW18 SW_SPST, SW19 SW_SPDT, SW2 SW_SPST, SW20 SW_SPST, SW21 SW_SPST, SW22 SW_SPST, SW23 SW_SPST, SW24 SW_SPST, SW25 SW_SPST, SW26 SW_SPST, SW27 SW_SPST, SW28 SW_SPST, SW29 SW_SPST, SW3 SW_SPST, SW30 SW_SPST, SW31 SW_SPST, SW32 SW_SPST, SW33 SW_SPST, SW34 SW_SPST, SW35 SW_SPST, SW36 SW_SPST, SW37 SW_SPST, SW38 SW_SPDT, SW4 SW_SPST, SW5 SW_SPST, SW6 SW_SPST, SW7 SW_SPST, SW8 SW_SPST, SW9 SW_SPST, U1 Seeeduino Xiao nRF52840, U2 Seeeduino Xiao nRF52840

Commit message: layout v1
Parts:
- moved D15 141.2 mm to (208.4, 140.7)
- moved D16 141.2 mm to (208.4, 144.0)
- moved D17 141.2 mm to (208.4, 147.4)
- moved D18 141.2 mm to (208.4, 150.7)
- moved D33 141.2 mm to (208.4, 63.5)
- moved D34 141.2 mm to (208.4, 66.9)
- moved D35 141.2 mm to (208.4, 70.2)
- moved D36 141.2 mm to (208.4, 73.6)
- moved H1 141.2 mm to (170.8, 142.0)
- moved H2 141.2 mm to (170.8, 147.9)
- moved H3 141.2 mm to (170.8, 153.9)
- moved H4 141.2 mm to (170.8, 159.8)
- moved H5 141.2 mm to (170.8, 64.8)
- moved H6 141.2 mm to (170.8, 70.8)
- moved H7 141.2 mm to (170.8, 76.7)
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
Commit message: new layout, new schematic, new footprints, new everything really
Parts:
- removed D1, D10, D11, D12, D13, D14, D15, D16, D17, D18, D19, D2, D20, D21, D22, D23, D24, D25, D26, D27, D28, D29, D3, D30, D31, D32, D33, D34, D35, D36, D4, D5, D6, D7, D8, D9: 1N4148W, Diode_SMD:D_SOD-123
- removed the H1 at (170.8, 142.0)
- removed H10, H11, H8: MountingHole, MountingHole:MountingHole_2.2mm_M2
- removed H13, H14, H7: MountingHole, Panelization:mouse-bite-5mm-slot
- removed the H2 at (170.8, 147.9)
- removed the H3 at (170.8, 153.9)
- removed the H4 at (170.8, 159.8)
- removed R1, R3: 2M, Resistor_SMD:R_0805_2012Metric
- removed R2, R4: 806k, Resistor_SMD:R_0805_2012Metric
- removed the SW1 at (176.4, 96.2)
- removed the SW10 at (227.7, 113.3)
- removed the SW11 at (244.9, 113.3)
- removed the SW12 at (262.0, 113.3)
- removed the SW13 at (176.4, 130.5)
- removed the SW14 at (193.5, 130.5)
- removed the SW15 at (210.6, 130.5)
- removed the SW16 at (227.7, 130.5)
- removed the SW17 at (244.9, 130.5)
- removed the SW18 at (262.0, 130.5)
- removed the SW19 at (219.1, 141.7)
- removed the SW2 at (193.5, 96.2)
- removed the SW3 at (210.6, 96.2)
- removed the SW4 at (227.7, 96.2)
- removed the SW5 at (244.9, 96.2)
- removed the SW6 at (262.0, 96.2)
- removed the SW7 at (176.4, 113.3)
- removed the SW8 at (193.5, 113.3)
- removed the SW9 at (210.6, 113.3)
- removed the TP1 at (213.3, 141.0)
- removed the TP2 at (213.3, 145.1)
- removed U2: Seeeduino Xiao nRF52840, nrf52840:modified-XIAO-nRF52840-SMD
- H1: renamed from H5; footprint Panelization:mouse-bite-5mm-slot -> MountingHole:MountingHole_2.2mm_M2
- H2: renamed from H12; footprint Panelization:mouse-bite-5mm-slot -> MountingHole:MountingHole_2.2mm_M2
- H4: renamed from H6; footprint Panelization:mouse-bite-5mm-slot -> MountingHole:MountingHole_2.2mm_M2
- SW19: renamed from SW38; footprint switch:SW-SMD_MSK12CO2 -> nrf52840:SW-SMD_MSK12CO2
- TP1: renamed from TP3; footprint TestPoint:TestPoint_Pad_D2.0mm -> TestPoint:TestPoint_Pad_2.5x2.5mm
- TP2: renamed from TP4; footprint TestPoint:TestPoint_Pad_D2.0mm -> TestPoint:TestPoint_Pad_2.5x2.5mm
- U1: value Seeeduino Xiao nRF52840 -> SuperMini nRF52840; footprint nrf52840:modified-XIAO-nRF52840-SMD -> keyboard_reversible:ProMicro_flipped
- moved U1 134.0 mm to (104.4, 43.8), turned to -90 degrees
- moved SW19 62.0 mm to (163.8, 92.5)
- moved H1 55.1 mm to (198.4, 112.5)
- moved H3 55.1 mm to (269.6, 114.7)
- moved H4 55.1 mm to (198.4, 118.4)
- moved H2 55.1 mm to (261.1, 114.9)
- moved TP1 55.1 mm to (240.9, 111.5)
- moved TP2 55.1 mm to (240.9, 115.6)
- renumbered H9 to H3, SW22 to SW1, SW25 to SW10, SW32 to SW11, SW33 to SW12, SW31 to SW13, SW34 to SW14, SW30 to SW15, SW35 to SW16, SW36 to SW17, SW37 to SW18, SW23 to SW2, SW21 to SW3, SW24 to SW4, SW20 to SW5, SW27 to SW6, SW28 to SW7, SW26 to SW8, SW29 to SW9
Connections:
- SW1 pad 1: /right/col2 -> unconnected-(SW1-A-Pad1)
- SW1 pad 2: Net-(D21-A) -> GND
- SW10 pad 1: /right/col0 -> unconnected-(SW10-A-Pad1)
- SW10 pad 2: Net-(D24-A) -> GND
- SW11 pad 1: /right/col2 -> unconnected-(SW11-A-Pad1)
- SW11 pad 2: Net-(D31-A) -> GND
- SW12 pad 1: /right/col3 -> unconnected-(SW12-A-Pad1)
- SW12 pad 2: Net-(D32-A) -> GND
- SW13 pad 1: /right/col1 -> unconnected-(SW13-A-Pad1)
- SW13 pad 2: Net-(D30-A) -> GND
- SW14 pad 1: /right/col4 -> unconnected-(SW14-A-Pad1)
- SW14 pad 2: Net-(D33-A) -> GND
- SW15 pad 1: /right/col0 -> unconnected-(SW15-A-Pad1)
- SW15 pad 2: Net-(D29-A) -> GND
- SW16 pad 1: /right/col2 -> unconnected-(SW16-A-Pad1)
- SW16 pad 2: Net-(D34-A) -> GND
- SW17 pad 1: /right/col3 -> unconnected-(SW17-A-Pad1)
- SW17 pad 2: Net-(D35-A) -> GND
- SW18 pad 1: /right/col4 -> unconnected-(SW18-A-Pad1)
- SW18 pad 2: Net-(D36-A) -> GND
- SW19 pad 1: Net-(SW38-A) -> unconnected-(SW19-A-Pad1)
- SW19 pad 2: Net-(SW38-B) -> Net-(SW19-B)
- SW19 pad 3: unconnected-(SW38-C-Pad3) -> Net-(SW19-C)
- SW2 pad 1: /right/col3 -> unconnected-(SW2-A-Pad1)
- SW2 pad 2: Net-(D22-A) -> GND
- SW3 pad 1: /right/col1 -> unconnected-(SW3-A-Pad1)
- SW3 pad 2: Net-(D20-A) -> GND
- SW4 pad 1: /right/col4 -> unconnected-(SW4-A-Pad1)
- SW4 pad 2: Net-(D23-A) -> GND
- SW5 pad 1: /right/col0 -> unconnected-(SW5-A-Pad1)
- SW5 pad 2: Net-(D19-A) -> GND
- SW6 pad 1: /right/col2 -> unconnected-(SW6-A-Pad1)
- SW6 pad 2: Net-(D26-A) -> GND
- SW7 pad 1: /right/col3 -> unconnected-(SW7-A-Pad1)
- SW7 pad 2: Net-(D27-A) -> GND
- SW8 pad 1: /right/col1 -> unconnected-(SW8-A-Pad1)
- SW8 pad 2: Net-(D25-A) -> GND
- SW9 pad 1: /right/col4 -> unconnected-(SW9-A-Pad1)
- SW9 pad 2: Net-(D28-A) -> GND
- TP1 pad 1: GND -> Net-(SW19-C)
- TP2 pad 1: Net-(SW38-A) -> GND
- U1 pad 1: /left/bt_pin -> unconnected-(U1-P0.06-Pad1)
- U1 pad 11: /left/row1 -> unconnected-(U1-P1.04-LF-Pad11)
- U1 pad 12: /left/row2 -> unconnected-(U1-P1.06-LF-Pad12)
- U1 pad 13: /left/row3 -> unconnected-(U1-BAT+-Pad13)
- U1 pad 14: unconnected-(U1-P1.12-Pad14) -> GND
- U1 pad 15: GND -> unconnected-(U1-RST-Pad15)
- U1 pad 16: Net-(SW19-B) -> unconnected-(U1-3V3-Pad16)
- U1 pad 2: /left/col0 -> unconnected-(U1-P0.08-Pad2)
- U1 pad 3: /left/col1 -> GND
- U1 pad 4: /left/col2 -> GND
- U1 pad 5: /left/col3 -> unconnected-(U1-P0.17-Pad5)
- U1 pad 6: /left/col4 -> unconnected-(U1-P0.20-Pad6)
- U1 pad 7: /left/row0 -> unconnected-(U1-P0.22-Pad7)
- U1 pad 9: GND -> unconnected-(U1-P1.00-Pad9)
