File: winglets.kicad_sch (KiCad schematic)
At the start: 0 parts

Commit message: footprints
Changed lines of the file:
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@@
 	(paper "A4")
 	(sheet
-		(at 121.92 33.02)
-		(size 60.96 44.45)
+		(at 142.24 66.04)
+		(size 66.04 33.02)
 		(exclude_from_sim no)
 		(in_bom yes)
@@
 		)
 		(property "Sheetname" "right"
-			(at 121.92 32.3084 0)
+			(at 142.24 65.3284 0)
 			(effects
 				(font
@@
 		)
 		(property "Sheetfile" "side.kicad_sch"
-			(at 121.92 78.0546 0)
+			(at 142.24 99.6446 0)
 			(effects
 				(font

Commit message: new layout, new schematic, new footprints, new everything really
Parts:
- added H1, H2, H3, H4: MountingHole, MountingHole:MountingHole_2.2mm_M2, symbol Mechanical:MountingHole
- added SW1, SW10, SW11, SW12, SW13, SW14, SW15, SW16, SW17, SW18, SW2, SW3, SW4, SW5, SW6, SW7, SW8, SW9: SW_SPST, lad1337:CPG1316S01D02_reversible, symbol Switch:SW_SPST
- added SW19: SW_SPDT, nrf52840:SW-SMD_MSK12CO2, symbol Switch:SW_SPDT
- added TP1, TP2: TestPoint, TestPoint:TestPoint_Pad_2.5x2.5mm, symbol Connector:TestPoint
- added U1: SuperMini nRF52840, keyboard_reversible:ProMicro_flipped, symbol PCM_marbastlib-promicroish:SuperMini_nRF52840
Connections:
- new net: SW19.2 (B), U1.29 (BAT+)
- new net: SW19.3 (C), TP1.1
- new net GND: SW1.2 (B), SW10.2 (B), SW11.2 (B), SW12.2 (B), SW13.2 (B), SW14.2 (B), SW15.2 (B), SW16.2 (B), SW17.2 (B), SW18.2 (B), SW2.2 (B), SW3.2 (B), SW4.2 (B), SW5.2 (B), SW6.2 (B), SW7.2 (B), SW8.2 (B), SW9.2 (B), TP2.1, U1.14 (GND), U1.28 (GND), U1.3 (GND), U1.4 (GND)
Other:
- removed sheet left
- removed sheet right
